File: E-throttle/E-throttle.kicad_pcb (KiCad board)
At the start: 2 copper layers, 125 x 70 mm, 34 parts, among them J1 PROG, J2 JTAG, J3 Conn_01x11, J4 Conn_01x11, J5 776087-1, Q1 NMOS, SW1 SW_Push, U1 ESP32-S3-WROOM-1-N16R8, U2 LM317_SOT-223, U3 LM317_SOT-223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

Commit message: Wiring completed
Parts:
- moved R14 138.6 mm to (200.7, 107.2)
- moved R4 138.6 mm to (200.7, 95.0)
- moved R5 138.6 mm to (200.7, 99.1)
- moved R13 138.6 mm to (200.7, 103.1)
- moved C5 108.7 mm to (188.5, 91.4)
- moved J3 101.2 mm to (196.8, 81.8)
- moved R10 98.3 mm to (200.7, 91.2)
- moved J1 93.2 mm to (191.3, 82.0)
- moved C2 72.4 mm to (144.5, 93.0), turned to -90 degrees
- moved J2 71.8 mm to (180.8, 90.2), turned to 180 degrees
- moved SW1 71.4 mm to (150.1, 100.8), turned to 180 degrees
- moved C1 70.9 mm to (149.1, 93.0), turned to -90 degrees
- moved C4 69.6 mm to (150.1, 107.2)
- moved C3 63.0 mm to (143.8, 107.2)
- moved U3 57.4 mm to (159.7, 120.4), turned to 180 degrees
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Routing:
- net GND: track 0.00 -> 316.7 mm, vias 0 -> 5
- net +5V: track 0.00 -> 181.7 mm
- net +3V3: track 0.00 -> 165.6 mm, vias 0 -> 2
- net /CAN-H: track 0.00 -> 113.1 mm, vias 0 -> 1
- net /CAN-L: track 0.00 -> 110.3 mm, vias 0 -> 2
- net +12V: track 0.00 -> 110.2 mm, vias 0 -> 4
- net /BLIP-IN: track 0.00 -> 92.4 mm, vias 0 -> 2
- net /APPS-SIG2-OUT: track 0.00 -> 76.7 mm, vias 0 -> 1
- net /APPS-SIG2: track 0.00 -> 73.6 mm, vias 0 -> 3
- net /BLIP-OUT: track 0.00 -> 66.5 mm, vias 0 -> 6
- net /DIAG0: track 0.00 -> 63.5 mm, vias 0 -> 3
- net /TPS-SIG1: track 0.00 -> 60.4 mm, vias 0 -> 1
- net /IDLE: track 0.00 -> 60.2 mm, vias 0 -> 1
- net /TPS-SIG2: track 0.00 -> 56.4 mm, vias 0 -> 4
- net /TPS-GND2: track 0.00 -> 52.4 mm, vias 0 -> 2
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Other:
- board size 125 x 70 mm -> 82.1 x 70 mm
