File: E-throttle/E-throttle.kicad_pcb (KiCad board)
At the start: 2 copper layers, 88.9 x 72.4 mm, 38 parts, among them J1 PROG, J2 JTAG, J3 Conn_01x11, J4 Conn_01x11, J5 776087-1, Q1 NMOS, SW1 SW_Push, U1 ESP32-S3-WROOM-1-N16R8, U2 LM317_SOT-223, U3 LM317_SOT-223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

Commit message: Add logo and attribution to PCB
Parts:
- added G***: LOGO, FBR_Footprints:FBR_Logo_.9in, B.Cu at (210.8, 105.4)
Other:
- board text added: "Designed by Nonthapat U and Clement Tong, Feb 2025"
